File: Schematics/ElectronicCompass_T05.sch (EAGLE design)
At the start: 46 parts, among them Q1 TP0604N3, Q2 TP0604N3, Q3 TP0604N3, Q4 TP0604N3, U1 ATMEGA32U4, X1 USBSMD

Commit message: Made it prettier...
Parts:
- added JP8: LCD Mount, pinhead:PINHD-1X8
- added TP15, TP16, TP17, TP19, TP20, TP21, TP22, TP23: TPTP06R, testpad:TPTP06R
- C10: value 10u -> 10uF
- C4: value 10uF -> 1uF
- JP1, JP2: value (none) -> To Sensor
- JP3: value (none) -> To LCD
Connections:
- new net N$28: JP8.7, TP22.TP
- new net N$29: JP8.6, TP21.TP
- new net N$30: JP8.5, TP20.TP
- new net N$31: JP8.4, TP19.TP
- new net N$32: JP8.3, TP17.TP
- new net N$33: JP8.2, TP16.TP
- new net N$35: JP8.1, TP15.TP
- new net N$37: C12.1, U1.UVCC, U1.VBUS, X1.VBUS
- net D/C: now also JP3.4
- net GND: now also JP2.3, JP3.6, JP3.7, Q1.S
- net INT1: now also JP2.1
- net INT2: now also JP2.2
- net LCD_BKLT: now also JP3.1
- net MOSI: now also JP3.3
- net N$10: now also JP8.8, TP23.TP; no longer C12.1, Q1.S, X1.VBUS
- net N$34: now also JP1.3
- net RESET: now also JP3.5
- net SCL: now also JP1.1
- net SCLK: now also JP3.2
- net SDA: now also JP1.2
- net VCC': now also JP2.4, JP3.8
Other:
- note added: "LCD Mounting/TP"
- note added: "LTC4067"
- moved on the sheet: C1, C4

Commit message: Added ON/OFF switch
Parts:
- added S2: ON/OFF, switch-dil:DS01E
Connections:
- new net N$36: C10.1, LTC4067.OUT, Q2.S, S2.1
- net VCC: now also S2.2; no longer C10.1, LTC4067.OUT, Q2.S
Changed lines of the file:
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@@
 <part name="TP23" library="testpad" deviceset="TP" device="TP06R"/>
 <part name="GND3" library="SparkFun" deviceset="GND" device=""/>
+<part name="S2" library="switch-dil" deviceset="DS01E" device="" value="ON/OFF"/>
 </parts>
 <sheets>
@@
 <instance part="G1" gate="G$1" x="88.9" y="40.64" rot="R90"/>
 <instance part="GND19" gate="1" x="88.9" y="33.02"/>
-<instance part="P+3" gate="VCC" x="119.38" y="63.5"/>
+<instance part="P+3" gate="VCC" x="127" y="63.5"/>
 <instance part="GND6" gate="1" x="111.76" y="48.26"/>
 <instance part="GND12" gate="1" x="86.36" y="-27.94"/>
@@
 <instance part="TP23" gate="G$1" x="231.14" y="-53.34" rot="R90"/>
 <instance part="GND3" gate="1" x="91.44" y="15.24"/>
+<instance part="S2" gate="1" x="119.38" y="55.88" rot="R270"/>
 </instances>
 <busses>
@@
 </segment>
 <segment>
-<pinref part="LTC4067" gate="G$1" pin="OUT"/>
-<pinref part="C10" gate="G$1" pin="1"/>
-<wire x1="68.58" y1="55.88" x2="86.36" y2="55.88" width="0.1524" layer="91"/>
-<wire x1="86.36" y1="55.88" x2="101.6" y2="55.88" width="0.1524" layer="91"/>
-<wire x1="101.6" y1="55.88" x2="119.38" y2="55.88" width="0.1524" layer="91"/>
-<junction x="101.6" y="55.88"/>
-<pinref part="Q2" gate="G$1" pin="S"/>
-<wire x1="81.28" y1="45.72" x2="86.36" y2="45.72" width="0.1524" layer="91"/>
-<wire x1="86.36" y1="45.72" x2="86.36" y2="55.88" width="0.1524" layer="91"/>
-<junction x="86.36" y="55.88"/>
-<pinref part="P+3" gate="VCC" pin="VCC"/>
-<wire x1="119.38" y1="55.88" x2="119.38" y2="60.96" width="0.1524" layer="91"/>
-</segment>
-<segment>
 <pinref part="Q4" gate="G$1" pin="S"/>
 <pinref part="P+4" gate="1" pin="VCC"/>
@@
 <wire x1="190.5" y1="-48.26" x2="190.5" y2="-22.86" width="0.1524" layer="91"/>
 <pinref part="P+6" gate="1" pin="VCC"/>
+</segment>
+<segment>
+<pinref part="P+3" gate="VCC" pin="VCC"/>
+<wire x1="127" y1="60.96" x2="127" y2="55.88" width="0.1524" layer="91"/>
+<pinref part="S2" gate="1" pin="2"/>
+<wire x1="127" y1="55.88" x2="124.46" y2="55.88" width="0.1524" layer="91"/>
 </segment>
 </net>
@@
 </segment>
 </net>
+<net name="N$36" class="0">
+<segment>
+<pinref part="LTC4067" gate="G$1" pin="OUT"/>
+<pinref part="C10" gate="G$1" pin="1"/>
+<wire x1="68.58" y1="55.88" x2="86.36" y2="55.88" width="0.1524" layer="91"/>
+<wire x1="86.36" y1="55.88" x2="101.6" y2="55.88" width="0.1524" layer="91"/>
+<wire x1="101.6" y1="55.88" x2="114.3" y2="55.88" width="0.1524" layer="91"/>
+<junction x="101.6" y="55.88"/>
+<pinref part="Q2" gate="G$1" pin="S"/>
+<wire x1="81.28" y1="45.72" x2="86.36" y2="45.72" width="0.1524" layer="91"/>
+<wire x1="86.36" y1="45.72" x2="86.36" y2="55.88" width="0.1524" layer="91"/>
+<junction x="86.36" y="55.88"/>
+<pinref part="S2" gate="1" pin="1"/>
+</segment>
+</net>

Commit message: The schematic has been finalized!
Parts:
- removed C1: 0.1uF, SparkFun:CAP0805
- removed LTC4067: LTC4067, LTC4067:LTC4067
- added C2: 10nF, rcl:C-USC0805
- added C3: 0.1uF, rcl:C-USC0805
- added TP24, TP25: TPTP06R, testpad:TPTP06R
- added U$1: LTC4067, LTC4067:LTC4067
- C11: value 10 uF -> 1uF
- C5: value 10nF -> 10uF
- Q1, Q2, Q3, Q4: value TP0604N3 -> SPB80P06P; device transistor-fet:TP0604N3 -> transistor-fet:SPB80P06P
Connections:
- removed net N$37: C12.1, U1.UVCC, U1.VBUS, X1.VBUS
- net AREF: now also C3.1; no longer C1.1
- net GND: now also C3.2, C5.2, U$1.GND, U$1.NTC; no longer C1.2, LTC4067.GND, LTC4067.NTC, Q1.S
- net INT1: now also U1.PF1(ADC1); no longer U1.PD2(RX)
- net INT2: now also U1.PF0(ADC0); no longer U1.PD3(TX)
- net N$1: now also R6.1, U$1.PROG; no longer C5.1, LTC4067.OVP, Q1.G
- net N$11: now also C11.1, C12.1, C2.1, Q1.S, U$1.OVI, U1.UVCC, U1.VBUS, X1.VBUS; no longer LTC4067.GATE, Q2.G
- net N$16: now also Q2.G, U$1.GATE; no longer C5.2, LTC4067.OVI
- net N$19: now also U1.PD2(RX); no longer U1.PF1(ADC1)
- net N$20: now also U1.PD3(TX); no longer U1.PF0(ADC0)
- net N$36: now also TP25.TP, U$1.OUT; no longer LTC4067.OUT
- net N$4: now also R4.2, U$1.CLPROG; no longer LTC4067.PROG, R6.1
- net N$5: now also TP24.TP, U$1.BAT; no longer LTC4067.BAT
- net N$6: now also C5.1, LED1.A, Q1.D, U$1.IN; no longer LTC4067.CLPROG, R4.2
- net N$7: now also R5.2, U$1.CHARGE; no longer LTC4067.CHARGE, R5.1
- net N$8: now also R5.1; no longer R5.2
- net N$9: now also C2.2, Q1.G, U$1.OVP; no longer C11.1, LED1.A, LTC4067.IN, Q1.D
- net VCC: now also U$1.ILIM0, U$1.ILIM1; no longer LTC4067.ILIM0, LTC4067.ILIM1
Other:
- note added: "4"
- note added: "LSM303DLM"
- note added: "Nokia 5110"
- note added: "Supply Voltage 3.3V"
- moved on the sheet: C10, C11, C5, G1, LED1, R4, R5, R6, R7, S2, TP5, TP6

Commit message: Last minute changes to schematic before the layout begins
Parts:
- added TP26, TP27, TP28: TPTP06R, testpad:TPTP06R
- C12: value 1uF -> 10uF
Connections:
- new net N$37: Q3.G, U1.PB0(SS)
- new net N$38: TP26.TP, U1.PC7
- new net N$40: TP28.TP, U1.PB3(MISO)
- net N$39: now also TP27.TP; no longer Q3.G
Other:
- moved on the sheet: JP3, Q3, Q4, R7, R8
