File: Schematics/ElectronicCompass_T05.brd (EAGLE design)
At the start: 50.5 x 50.8 mm, 64 parts, among them Q1 FDN360P, Q2 FDN360P, Q3 FDN360P, Q4 FDN360P, Q5 BC817-16LT1SMD, Q6 BC817-16LT1SMD, U1 ATMEGA32U4, X1 USBSMD, Y1 16MHz

Commit message: sch changes
Parts:
- removed S2: ON/OFF, switch-dil:DS-01
- added JP5: ON/OFF, pinhead:1X02
Connections:
- removed net N$11: C7.2, U1.14, U1.24, U1.34, U1.44
- net GND: now also C7.2
- net N$36: now also JP5.1; no longer S2.1
- net VCC: now also JP5.2, U1.14, U1.24, U1.34, U1.44; no longer S2.2
Routing:
- net N$36: track 45.8 -> 20.0 mm
- net N$11: track 17.2 -> 0.00 mm
- net VCC: track 58.6 -> 54.9 mm, vias 3 -> 2
Changed lines of the file:
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@@
 <attribute name="TP_SIGNAL_NAME" value="" x="8.255" y="49.53" size="1.778" layer="28" rot="MR180" display="off"/>
-</element>
-<element name="S2" library="switch-dil" package="DS-01" value="ON/OFF" x="7.62" y="43.815" rot="MR270">
-<attribute name="OC_NEWARK" value="unknown" x="7.62" y="43.815" size="1.778" layer="28" rot="MR270" display="off"/>
-<attribute name="MPN" value="" x="7.62" y="43.815" size="1.778" layer="28" rot="MR270" display="off"/>
-<attribute name="MF" value="" x="7.62" y="43.815" size="1.778" layer="28" rot="MR270" display="off"/>
-<attribute name="OC_FARNELL" value="unknown" x="7.62" y="43.815" size="1.778" layer="28" rot="MR270" display="off"/>
 </element>
 <element name="TP24" library="testpad" package="TP06R" value="TPTP06R" x="43.815" y="49.53" rot="MR180">
@@
 <element name="Q5" library="transistor-npn" package="SOT23-BEC" value="BC817-16LT1SMD" x="2.25" y="-26.75"/>
 <element name="Q6" library="transistor-npn" package="SOT23-BEC" value="BC817-16LT1SMD" x="2.25" y="-34.05"/>
+<element name="JP5" library="pinhead" package="1X02" value="ON/OFF" x="2.95" y="-41.3"/>
 </elements>
 <signals>
-<signal name="GND" airwireshidden="yes">
+<signal name="GND">
 <contactref element="S1" pad="1"/>
 <contactref element="X1" pad="GND"/>
@@
 <contactref element="Q5" pad="E"/>
 <contactref element="Q6" pad="E"/>
+<contactref element="C7" pad="2"/>
 <wire x1="35.875" y1="40.005" x2="44.45" y2="44.45" width="0" layer="19" extent="1-1"/>
 <wire x1="30.48" y1="36.83" x2="35.875" y2="40.005" width="0" layer="19" extent="1-1"/>
@@
 <wire x1="6.985" y1="15.875" x2="5.2" y2="8.82" width="0" layer="19" extent="16-16"/>
 <wire x1="8.85" y1="19.355" x2="6.985" y2="15.875" width="0" layer="19" extent="1-16"/>
-<wire x1="0.955" y1="-14.76375" x2="12.385" y2="3.33375" width="0" layer="19" extent="1-16"/>
+<wire x1="2.855" y1="-3.33375" x2="12.385" y2="3.33375" width="0" layer="19" extent="1-16"/>
+<wire x1="0.955" y1="-14.76375" x2="2.855" y2="-3.33375" width="0" layer="19" extent="1-1"/>
 <wire x1="3.2" y1="-27.85" x2="0.955" y2="-14.76375" width="0" layer="19" extent="1-1"/>
 <wire x1="3.2" y1="-35.15" x2="3.2" y2="-27.85" width="0" layer="19" extent="1-1"/>
@@
 <signal name="VCC">
 <contactref element="R1" pad="2"/>
-<contactref element="S2" pad="2"/>
 <contactref element="Q4" pad="2"/>
 <wire x1="44.28" y1="7.45" x2="44.45" y2="7.46125" width="0.254" layer="16"/>
@@
 <wire x1="22.225" y1="19.685" x2="20.955" y2="19.20875" width="0.3048" layer="1"/>
 <via x="20.955" y="19.20875" extent="1-16" drill="0.6"/>
-<wire x1="3.81" y1="43.815" x2="7.3025" y2="43.815" width="0.254" layer="16"/>
-<wire x1="7.3025" y1="43.815" x2="9.8425" y2="41.91" width="0.254" layer="16"/>
-<wire x1="9.8425" y1="41.91" x2="12.7" y2="41.91" width="0.254" layer="16"/>
-<wire x1="12.7" y1="41.91" x2="13.81125" y2="43.18" width="0.254" layer="16"/>
-<wire x1="13.81125" y1="43.18" x2="15.875" y2="43.18" width="0.254" layer="16"/>
-<wire x1="15.875" y1="43.18" x2="17.145" y2="41.5925" width="0.254" layer="16"/>
-<wire x1="18.8" y1="36.73875" x2="17.62125" y2="37.94125" width="0.254" layer="1"/>
-<wire x1="17.145" y1="41.5925" x2="17.4625" y2="41.275" width="0.254" layer="16"/>
-<wire x1="17.4625" y1="41.275" x2="17.62125" y2="37.94125" width="0.254" layer="16"/>
-<via x="17.62125" y="37.94125" extent="1-16" drill="0.6"/>
-<contactref element="C7" pad="1"/>
 <contactref element="Q3" pad="2"/>
 <contactref element="R7" pad="2"/>
 <contactref element="R10" pad="1"/>
+<contactref element="JP5" pad="2"/>
+<contactref element="U1" pad="14"/>
+<contactref element="U1" pad="34"/>
+<contactref element="U1" pad="24"/>
+<contactref element="U1" pad="44"/>
+<wire x1="23.535" y1="18.79875" x2="23.535" y2="17.89875" width="0.254" layer="1"/>
+<wire x1="23.535" y1="17.89875" x2="24.765" y2="16.98625" width="0.254" layer="1"/>
+<wire x1="24.765" y1="16.98625" x2="27.94" y2="16.98625" width="0.254" layer="1"/>
+<wire x1="28.525" y1="18.6" x2="28.535" y2="18.79875" width="0.254" layer="1"/>
+<wire x1="28.525" y1="18.6" x2="28.525" y2="17.93875" width="0.254" layer="1"/>
+<wire x1="28.525" y1="17.93875" x2="27.94" y2="16.98625" width="0.254" layer="1"/>
+<wire x1="29.435" y1="13.39875" x2="28.82875" y2="13.39875" width="0.254" layer="1"/>
+<wire x1="28.82875" y1="13.39875" x2="27.78125" y2="14.2875" width="0.254" layer="1"/>
+<wire x1="27.78125" y1="14.2875" x2="27.94" y2="16.98625" width="0.254" layer="1"/>
+<wire x1="24.535" y1="11.99875" x2="24.535" y2="12.7875" width="0.254" layer="1"/>
+<wire x1="24.535" y1="12.7875" x2="25.7175" y2="14.44625" width="0.254" layer="1"/>
+<wire x1="25.7175" y1="14.44625" x2="27.78125" y2="14.2875" width="0.254" layer="1"/>
+<contactref element="C7" pad="1"/>
 <wire x1="42.86" y1="7.45" x2="44.28" y2="7.45" width="0" layer="19" extent="16-16"/>
-<wire x1="23.01875" y1="19.48625" x2="42.86" y2="7.45" width="0" layer="19" extent="1-16"/>
-<wire x1="18.8" y1="36.73875" x2="24.65" y2="36.08" width="0" layer="19" extent="1-1"/>
+<wire x1="29.435" y1="13.39875" x2="42.86" y2="7.45" width="0" layer="19" extent="1-16"/>
+<wire x1="23.01875" y1="19.48625" x2="23.535" y2="18.79875" width="0" layer="19" extent="1-1"/>
 <wire x1="0.955" y1="-3.33375" x2="10.63625" y2="13.9675" width="0" layer="19" extent="1-16"/>
 <wire x1="2.855" y1="-9.2075" x2="0.955" y2="-3.33375" width="0" layer="19" extent="1-1"/>
 <wire x1="0.955" y1="-20.32" x2="2.855" y2="-9.2075" width="0" layer="19" extent="1-1"/>
+<wire x1="4.22" y1="-41.3" x2="0.955" y2="-20.32" width="0" layer="19" extent="1-1"/>
 </signal>
 <signal name="UCAP">
@@
 <contactref element="Q2" pad="2"/>
 <contactref element="TP25" pad="TP"/>
-<contactref element="S2" pad="1"/>
 <contactref element="C10" pad="1"/>
 <contactref element="U$1" pad="P11"/>
 <wire x1="3.81" y1="49.53" x2="5.715" y2="49.53" width="0.254" layer="16"/>
-<wire x1="5.715" y1="49.53" x2="11.43" y2="43.815" width="0.254" layer="16"/>
-<wire x1="11.43" y1="43.815" x2="29.21" y2="43.815" width="0.254" layer="16"/>
 <wire x1="29.21" y1="43.815" x2="30.7975" y2="42.2275" width="0.254" layer="16"/>
 <wire x1="33.975" y1="40.005" x2="33.02" y2="40.005" width="0.254" layer="1"/>
@@
 <wire x1="33.9725" y1="40.0025" x2="33.975" y2="40.005" width="0.254" layer="1"/>
 <via x="30.7975" y="42.2275" extent="1-16" drill="0.6"/>
+<contactref element="JP5" pad="1"/>
+<wire x1="5.715" y1="49.53" x2="29.21" y2="43.815" width="0" layer="19" extent="16-16"/>
+<wire x1="1.68" y1="-41.3" x2="31.957" y2="37.58" width="0" layer="19" extent="1-1"/>
 </signal>
 <signal name="N$37">
@@
 <wire x1="35.245" y1="33.655" x2="31.957" y2="36.08" width="0" layer="19" extent="1-1"/>
 </signal>
-<signal name="N$11">
-<contactref element="U1" pad="14"/>
-<contactref element="U1" pad="34"/>
-<contactref element="U1" pad="24"/>
-<contactref element="U1" pad="44"/>
-<wire x1="23.535" y1="18.79875" x2="23.535" y2="17.89875" width="0.254" layer="1"/>
-<wire x1="23.535" y1="17.89875" x2="24.765" y2="16.98625" width="0.254" layer="1"/>
-<wire x1="24.765" y1="16.98625" x2="27.94" y2="16.98625" width="0.254" layer="1"/>
-<wire x1="28.525" y1="18.6" x2="28.535" y2="18.79875" width="0.254" layer="1"/>
-<wire x1="28.525" y1="18.6" x2="28.525" y2="17.93875" width="0.254" layer="1"/>
-<wire x1="28.525" y1="17.93875" x2="27.94" y2="16.98625" width="0.254" layer="1"/>
-<wire x1="29.435" y1="13.39875" x2="28.82875" y2="13.39875" width="0.254" layer="1"/>
-<wire x1="28.82875" y1="13.39875" x2="27.78125" y2="14.2875" width="0.254" layer="1"/>
-<wire x1="27.78125" y1="14.2875" x2="27.94" y2="16.98625" width="0.254" layer="1"/>
-<wire x1="24.535" y1="11.99875" x2="24.535" y2="12.7875" width="0.254" layer="1"/>
-<wire x1="24.535" y1="12.7875" x2="25.7175" y2="14.44625" width="0.254" layer="1"/>
-<wire x1="25.7175" y1="14.44625" x2="27.78125" y2="14.2875" width="0.254" layer="1"/>
-<contactref element="C7" pad="2"/>
-<wire x1="2.855" y1="-3.33375" x2="24.535" y2="11.99875" width="0" layer="19" extent="1-1"/>
-</signal>
 <signal name="N$38">

Commit message: New components
Parts:
- moved JP5 87.1 mm to (3.05, 45.8), turned to 270 degrees
- moved Q6 54.9 mm to (43.3, 2.35)
- moved Q5 46.7 mm to (38.7, 2.45)
- moved R10 38.6 mm to (33.3, 2.25), turned to 90 degrees
- moved R9 31.8 mm to (28.8, 2.19), turned to 270 degrees
- moved R7 25.7 mm to (24.9, 2.35), turned to 90 degrees
- moved C7 12.2 mm to (8.37, 7.04), turned to 270 degrees
Routing:
- net N$34: track 0.00 -> 8.94 mm
- net N$38: track 0.00 -> 6.19 mm
- net N$43: track 5.38 -> 0.00 mm
- net GND: track 1.81 -> 5.56 mm
- net VCC: track 54.9 -> 56.2 mm

Commit message: sch changes
Parts:
- added C8: 1uF, rcl:C0805
- added R11: 10k, resistor:M0805
- added S2: Switch, switch-dil:DS-01
Connections:
- new net N$11: C8.1, R11.1, S2.2, U1.33
- net GND: now also C8.2, S2.1; no longer U1.33
- net VCC: now also R11.2
Changed lines of the file:
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@@
 <element name="Q6" library="transistor-npn" package="SOT23-BEC" value="BC817-16LT1SMD" x="43.3" y="2.35"/>
 <element name="JP5" library="pinhead" package="1X02" value="ON/OFF" x="3.05" y="45.8" rot="R270"/>
+<element name="S2" library="switch-dil" package="DS-01" value="Switch" x="-6.25" y="5.95">
+<attribute name="OC_NEWARK" value="unknown" x="-6.25" y="5.95" size="1.778" layer="27" display="off"/>
+<attribute name="MPN" value="" x="-6.25" y="5.95" size="1.778" layer="27" display="off"/>
+<attribute name="MF" value="" x="-6.25" y="5.95" size="1.778" layer="27" display="off"/>
+<attribute name="OC_FARNELL" value="unknown" x="-6.25" y="5.95" size="1.778" layer="27" display="off"/>
+</element>
+<element name="C8" library="rcl" package="C0805" value="1uF" x="-6.75" y="-4.3"/>
+<element name="R11" library="resistor" package="M0805" value="10k" x="-6.75" y="-10.1"/>
 </elements>
 <signals>
@@
 <contactref element="U1" pad="15"/>
 <contactref element="U1" pad="5"/>
-<contactref element="U1" pad="33"/>
 <contactref element="C10" pad="2"/>
 <contactref element="R6" pad="2"/>
@@
 <wire x1="22.635" y1="15.89875" x2="23.51875" y2="15.89875" width="0.254" layer="1"/>
 <wire x1="23.51875" y1="15.89875" x2="23.65375" y2="16.03375" width="0.254" layer="1"/>
-<wire x1="25.0325" y1="12.22375" x2="25.035" y2="11.99875" width="0" layer="19" extent="1-1"/>
+<contactref element="C8" pad="2"/>
+<contactref element="S2" pad="1"/>
+<wire x1="35.875" y1="40.005" x2="44.45" y2="44.45" width="0" layer="19" extent="1-1"/>
+<wire x1="30.48" y1="36.83" x2="35.875" y2="40.005" width="0" layer="19" extent="1-1"/>
+<wire x1="29.003" y1="36.58" x2="30.48" y2="36.83" width="0" layer="19" extent="1-1"/>
+<wire x1="29.003" y1="36.08" x2="29.003" y2="36.58" width="0" layer="19" extent="1-1"/>
+<wire x1="29.003" y1="37.08" x2="29.003" y2="36.58" width="0" layer="19" extent="1-1"/>
+<wire x1="27.305" y1="40.325" x2="29.003" y2="37.08" width="0" layer="19" extent="1-1"/>
+<wire x1="22.225" y1="40.955" x2="27.305" y2="40.325" width="0" layer="19" extent="1-1"/>
+<wire x1="37.145" y1="33.655" x2="35.875" y2="40.005" width="0" layer="19" extent="1-1"/>
+<wire x1="39.37" y1="26.67" x2="37.145" y2="33.655" width="0" layer="19" extent="1-1"/>
+<wire x1="13.65" y1="32.7025" x2="22.225" y2="40.955" width="0" layer="19" extent="1-1"/>
+<wire x1="6.3525" y1="33.9725" x2="13.65" y2="32.7025" width="0" layer="19" extent="1-1"/>
+<wire x1="22.0675" y1="25.85125" x2="13.65" y2="32.7025" width="0" layer="19" extent="1-1"/>
+<wire x1="24.035" y1="18.79875" x2="22.0675" y2="25.85125" width="0" layer="19" extent="1-1"/>
+<wire x1="27.6225" y1="17.62125" x2="25.55875" y2="17.78" width="0" layer="19" extent="1-1"/>
+<wire x1="23.65375" y1="16.03375" x2="24.035" y2="18.065" width="0" layer="19" extent="1-1"/>
+<wire x1="25.0325" y1="12.7" x2="23.51875" y2="15.89875" width="0" layer="19" extent="1-1"/>
+<wire x1="25.035" y1="11.99875" x2="25.0325" y2="12.22375" width="0" layer="19" extent="1-1"/>
 <wire x1="27.46375" y1="13.335" x2="25.24125" y2="12.7" width="0" layer="19" extent="1-1"/>
-<wire x1="29.003" y1="37.08" x2="30.48" y2="36.83" width="0" layer="19" extent="1-1"/>
-<wire x1="35.875" y1="40.005" x2="30.48" y2="36.83" width="0" layer="19" extent="1-1"/>
+<wire x1="29.435" y1="12.89875" x2="27.46375" y2="13.335" width="0" layer="19" extent="1-1"/>
+<wire x1="16.98875" y1="14.9225" x2="22.635" y2="15.89875" width="0" layer="19" extent="1-1"/>
+<wire x1="16.66875" y1="9.98625" x2="16.98875" y2="14.9225" width="0" layer="19" extent="1-1"/>
+<wire x1="12.3975" y1="6.19125" x2="16.66875" y2="9.98625" width="0" layer="19" extent="1-1"/>
+<wire x1="12.385" y1="3.33375" x2="12.3975" y2="6.19125" width="0" layer="19" extent="1-16"/>
+<wire x1="8.36625" y1="6.095" x2="12.3975" y2="6.19125" width="0" layer="19" extent="1-1"/>
+<wire x1="5.2" y1="8.82" x2="8.36625" y2="6.095" width="0" layer="19" extent="1-1"/>
+<wire x1="29.21" y1="6.35" x2="29.435" y2="12.89875" width="0" layer="19" extent="1-1"/>
+<wire x1="31.75" y1="6.35" x2="29.21" y2="6.35" width="0" layer="19" extent="1-1"/>
+<wire x1="28.78625" y1="3.145" x2="29.21" y2="6.35" width="0" layer="19" extent="1-1"/>
+<wire x1="6.985" y1="15.875" x2="5.2" y2="8.82" width="0" layer="19" extent="16-16"/>
+<wire x1="8.85" y1="19.355" x2="6.985" y2="15.875" width="0" layer="19" extent="1-16"/>
+<wire x1="39.65" y1="1.35" x2="31.75" y2="6.35" width="0" layer="19" extent="1-1"/>
+<wire x1="44.25" y1="1.25" x2="39.65" y2="1.35" width="0" layer="19" extent="1-1"/>
+<wire x1="-6.25" y1="2.14" x2="5.2" y2="8.82" width="0" layer="19" extent="1-1"/>
+<wire x1="-5.8" y1="-4.3" x2="-6.25" y2="2.14" width="0" layer="19" extent="1-1"/>
 </signal>
 <signal name="VCC">
@@
 <wire x1="23.55" y1="19.55" x2="23.0425" y2="19.55" width="0.254" layer="1"/>
 <wire x1="23.0425" y1="19.55" x2="23.01875" y2="19.52625" width="0.254" layer="1"/>
+<contactref element="R11" pad="2"/>
 <wire x1="42.86" y1="7.45" x2="44.28" y2="7.45" width="0" layer="19" extent="16-16"/>
 <wire x1="33.27" y1="1.305" x2="42.86" y2="7.45" width="0" layer="19" extent="1-16"/>
@@
 <wire x1="8.36625" y1="7.995" x2="10.63625" y2="13.9675" width="0" layer="19" extent="1-16"/>
 <wire x1="3.05" y1="44.53" x2="17.145" y2="30.32125" width="0" layer="19" extent="1-1"/>
+<wire x1="-5.8" y1="-10.1" x2="8.36625" y2="7.995" width="0" layer="19" extent="1-1"/>
 </signal>
 <signal name="UCAP">
@@
 <wire x1="42.35" y1="1.25" x2="29.435" y2="16.39875" width="0" layer="19" extent="1-1"/>
 </signal>
+<signal name="N$11">
+<contactref element="U1" pad="33"/>
+<contactref element="S2" pad="2"/>
+<contactref element="C8" pad="1"/>
+<contactref element="R11" pad="1"/>
+<wire x1="-6.25" y1="9.76" x2="29.435" y2="17.89875" width="0" layer="19" extent="1-1"/>
+<wire x1="-7.7" y1="-4.3" x2="-6.25" y2="9.76" width="0" layer="19" extent="1-1"/>
+<wire x1="-7.7" y1="-10.1" x2="-7.7" y2="-4.3" width="0" layer="19" extent="1-1"/>
+</signal>
 </signals>
