File: Schematics/ElectronicCompass_T05.brd (EAGLE design)
At the start: 50.5 x 50.8 mm, 67 parts, among them Q1 FDN360P, Q2 FDN360P, Q3 FDN360P, Q4 FDN360P, Q5 BC817-16LT1SMD, Q6 BC817-16LT1SMD, U1 ATMEGA32U4, X1 USBSMD, Y1 16MHz

Commit message: sch update
Parts:
- removed JP5: ON/OFF, pinhead:1X02
- added S3: Off/On, switch-dil:DS-01
- S2: value Switch -> Pgm/Run
Connections:
- net N$36: now also S3.1; no longer JP5.1
- net VCC: now also S3.2; no longer JP5.2
Changed lines of the file:
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@@
 <element name="Q5" library="transistor-npn" package="SOT23-BEC" value="BC817-16LT1SMD" x="38.7" y="2.45"/>
 <element name="Q6" library="transistor-npn" package="SOT23-BEC" value="BC817-16LT1SMD" x="43.3" y="2.35"/>
-<element name="JP5" library="pinhead" package="1X02" value="ON/OFF" x="3.05" y="45.8" rot="R270"/>
-<element name="S2" library="switch-dil" package="DS-01" value="Switch" x="-6.25" y="5.95">
+<element name="S2" library="switch-dil" package="DS-01" value="Pgm/Run" x="-6.25" y="5.95">
 <attribute name="OC_NEWARK" value="unknown" x="-6.25" y="5.95" size="1.778" layer="27" display="off"/>
 <attribute name="MPN" value="" x="-6.25" y="5.95" size="1.778" layer="27" display="off"/>
@@
 <element name="C8" library="rcl" package="C0805" value="1uF" x="-6.75" y="-4.3"/>
 <element name="R11" library="resistor" package="M0805" value="10k" x="-6.75" y="-10.1"/>
+<element name="S3" library="switch-dil" package="DS-01" value="Off/On" x="-14.4" y="-5.65">
+<attribute name="OC_NEWARK" value="unknown" x="-14.4" y="-5.65" size="1.778" layer="27" display="off"/>
+<attribute name="MPN" value="" x="-14.4" y="-5.65" size="1.778" layer="27" display="off"/>
+<attribute name="MF" value="" x="-14.4" y="-5.65" size="1.778" layer="27" display="off"/>
+<attribute name="OC_FARNELL" value="unknown" x="-14.4" y="-5.65" size="1.778" layer="27" display="off"/>
+</element>
 </elements>
 <signals>
@@
 <contactref element="R7" pad="2"/>
 <contactref element="R10" pad="1"/>
-<contactref element="JP5" pad="2"/>
 <contactref element="U1" pad="14"/>
 <contactref element="U1" pad="34"/>
@@
 <wire x1="23.0425" y1="19.55" x2="23.01875" y2="19.52625" width="0.254" layer="1"/>
 <contactref element="R11" pad="2"/>
+<contactref element="S3" pad="2"/>
 <wire x1="42.86" y1="7.45" x2="44.28" y2="7.45" width="0" layer="19" extent="16-16"/>
 <wire x1="33.27" y1="1.305" x2="42.86" y2="7.45" width="0" layer="19" extent="1-16"/>
@@
 <wire x1="24.535" y1="11.99875" x2="24.9075" y2="3.305" width="0" layer="19" extent="1-1"/>
 <wire x1="8.36625" y1="7.995" x2="10.63625" y2="13.9675" width="0" layer="19" extent="1-16"/>
-<wire x1="3.05" y1="44.53" x2="17.145" y2="30.32125" width="0" layer="19" extent="1-1"/>
 <wire x1="-5.8" y1="-10.1" x2="8.36625" y2="7.995" width="0" layer="19" extent="1-1"/>
+<wire x1="-14.4" y1="-1.84" x2="-5.8" y2="-10.1" width="0" layer="19" extent="1-1"/>
 </signal>
 <signal name="UCAP">
@@
 <wire x1="33.9725" y1="40.0025" x2="33.975" y2="40.005" width="0.254" layer="1"/>
 <via x="30.7975" y="42.2275" extent="1-16" drill="0.6"/>
-<contactref element="JP5" pad="1"/>
+<contactref element="S3" pad="1"/>
 <wire x1="5.715" y1="49.53" x2="29.21" y2="43.815" width="0" layer="19" extent="16-16"/>
-<wire x1="3.05" y1="47.07" x2="3.81" y2="49.53" width="0" layer="19" extent="16-16"/>
+<wire x1="-14.4" y1="-9.46" x2="3.81" y2="49.53" width="0" layer="19" extent="16-16"/>
 </signal>
 <signal name="N$37">

Commit message: sch and layout changes
Parts:
- moved S3 53.8 mm to (6.15, 44.0), flipped to the bottom, turned to 90 degrees
- moved C8 53.3 mm to (40.3, 20.8), turned to 270 degrees
- moved R11 52.5 mm to (23.4, 32.9), turned to 180 degrees
- moved S2 49.0 mm to (40.4, 21.1), flipped to the bottom, turned to 90 degrees
- moved R9 42.3 mm to (45.9, 40.9), turned to 0 degrees
- moved JP4 40.9 mm to (35.6, 35.0), turned to 270 degrees
- moved Q5 30.1 mm to (12.7, 17.5), turned to 180 degrees
- moved TP28 21.8 mm to (1.05, 27.4), turned to 90 degrees
- moved TP11 20.7 mm to (1.26, 24.7), turned to 90 degrees
- moved C11 18.5 mm to (25.5, 36.9), turned to 0 degrees
- moved R10 16.4 mm to (19.1, 10.5), turned to 270 degrees
- moved C6 15.4 mm to (26.5, 10.7)
- moved C7 15.4 mm to (21.6, 14.9), turned to 90 degrees
- moved C1 15.2 mm to (31.5, 13.7)
- moved Y1 15.0 mm to (27.7, 13.3)
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Routing:
- net VCC': track 1.56 -> 48.3 mm
- net INT2: track 39.3 -> 0.00 mm
- net INT1: track 34.7 -> 0.00 mm, vias 1 -> 0
- net N$36: track 20.0 -> 49.4 mm
- net D/C: track 27.6 -> 0.00 mm, vias 2 -> 0
- net N$5: track 50.6 -> 25.5 mm, vias 2 -> 1
- net N$19: track 24.0 -> 0.00 mm, vias 1 -> 0
- net N$39: track 22.6 -> 0.00 mm, vias 1 -> 0
- net N$20: track 22.5 -> 0.00 mm, vias 1 -> 0
- net N$23: track 21.6 -> 0.00 mm, vias 1 -> 0
- net N$22: track 21.6 -> 0.00 mm, vias 1 -> 0
- net RESET: track 21.4 -> 0.00 mm, vias 2 -> 0
- net N$3: track 20.5 -> 0.00 mm, vias 1 -> 0
- net N$21: track 19.6 -> 0.00 mm, vias 1 -> 0
- net N$37: track 26.3 -> 8.91 mm, vias 1 -> 0
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
Commit message: layout done
Parts:
- moved TP4 24.7 mm to (49.2, 37.2)
- moved TP3 21.5 mm to (49.1, 34.4)
- moved TP10 20.5 mm to (1.54, 33.8), flipped to the bottom
- moved TP2 19.9 mm to (49.1, 31.4)
- moved TP1 14.2 mm to (49.1, 25.3)
- moved TP26 12.5 mm to (49.2, 22.6)
- moved C8 10.3 mm to (31.1, 25.4), turned to 90 degrees
- moved TP27 7.90 mm to (49.2, 5.43)
- moved S1 6.81 mm to (4.79, 7.17)
- moved TP11 6.62 mm to (1.47, 31.3), turned to 180 degrees
- moved TP6 4.71 mm to (49.2, 7.37)
- moved TP18 4.23 mm to (49.1, 28.6), turned to 0 degrees
- moved TP7 3.86 mm to (49.0, 11.6)
- moved R8 3.34 mm to (12.7, 9.42), turned to 0 degrees
- moved TP12 2.56 mm to (49.1, 14.3)
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Routing:
- net VCC: track 46.0 -> 92.1 mm, vias 2 -> 5
- net LCD_BKLT: track 3.33 -> 41.5 mm, vias 0 -> 2
- net GND: track 1.58 -> 38.5 mm, vias 0 -> 14
- net INT1: track 0.00 -> 36.5 mm, vias 0 -> 1
- net INT2: track 0.00 -> 36.3 mm, vias 0 -> 1
- net N$11: track 0.00 -> 33.2 mm
- net N$45: track 0.00 -> 31.8 mm
- net N$18: track 0.00 -> 30.8 mm, vias 0 -> 1
- net N$39: track 0.00 -> 28.5 mm, vias 0 -> 1
- net N$17: track 0.00 -> 28.3 mm, vias 0 -> 1
- net N$20: track 0.00 -> 27.6 mm, vias 0 -> 1
- net N$19: track 0.00 -> 27.4 mm, vias 0 -> 1
- net N$14: track 0.00 -> 26.3 mm, vias 0 -> 1
- net N$25: track 5.17 -> 31.3 mm, vias 0 -> 1
- net N$15: track 0.00 -> 26.0 mm, vias 0 -> 1
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
Commit message: layout update
Parts:
- moved R9 0.10 mm to (46.0, 40.9)
Routing:
- net VCC': track 48.3 -> 49.0 mm
Changed lines of the file:
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@@
 <attribute name="VALUE" x="23.511" y="13.6935" size="0.8128" layer="27" rot="R180"/>
 </element>
-<element name="R9" library="resistor" package="M0805" value="1k" x="45.855" y="40.88625" smashed="yes">
-<attribute name="NAME" x="44.839" y="41.90225" size="0.8128" layer="25"/>
-<attribute name="VALUE" x="44.839" y="38.60025" size="0.8128" layer="27"/>
+<element name="R9" library="resistor" package="M0805" value="1k" x="45.955" y="40.88625" smashed="yes">
+<attribute name="NAME" x="44.939" y="41.90225" size="0.8128" layer="25"/>
+<attribute name="VALUE" x="44.939" y="38.60025" size="0.8128" layer="27"/>
 </element>
 <element name="R10" library="resistor" package="M0805" value="1M" x="19.18" y="10.495" smashed="yes" rot="R270">
@@
 <contactref element="R9" pad="2"/>
 <contactref element="Q3" pad="3"/>
-<wire x1="34.29" y1="6.35" x2="39.31" y2="6.35" width="0.254" layer="1"/>
+<wire x1="34.29" y1="6.35" x2="39.31" y2="6.35" width="0.4064" layer="1"/>
 <wire x1="39.31" y1="6.35" x2="39.35" y2="6.36" width="0.254" layer="1"/>
-<wire x1="39.31" y1="6.35" x2="40.6" y2="6.35" width="0.254" layer="1"/>
-<wire x1="40.6" y1="6.35" x2="48.2" y2="13.95" width="0.254" layer="1"/>
-<wire x1="46.99" y1="44.45" x2="46.99" y2="41.07125" width="0.254" layer="1"/>
-<wire x1="46.99" y1="41.07125" x2="46.805" y2="40.88625" width="0.254" layer="1"/>
-<wire x1="46.805" y1="40.88625" x2="46.805" y2="37.895" width="0.254" layer="1"/>
-<wire x1="46.805" y1="37.895" x2="48.2" y2="36.5" width="0.254" layer="1"/>
-<wire x1="48.2" y1="36.5" x2="48.2" y2="13.95" width="0.254" layer="1"/>
+<wire x1="39.31" y1="6.35" x2="40.6" y2="6.35" width="0.6096" layer="1"/>
+<wire x1="40.6" y1="6.35" x2="48.85" y2="13.65" width="0.6096" layer="1"/>
+<wire x1="46.99" y1="44.45" x2="46.99" y2="41.07125" width="0.6096" layer="1"/>
+<wire x1="46.99" y1="41.07125" x2="46.905" y2="40.88625" width="0.254" layer="1"/>
+<wire x1="46.905" y1="40.88625" x2="46.905" y2="37.995" width="0.6096" layer="1"/>
+<wire x1="46.905" y1="37.995" x2="48.85" y2="36.2" width="0.6096" layer="1"/>
+<wire x1="48.85" y1="36.2" x2="48.85" y2="13.65" width="0.6096" layer="1"/>
 </signal>
 <signal name="RESET">

Commit message: staples
Routing:
- net GND: vias 14 -> 51
Changed lines of the file:
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@@
 <via x="45.05" y="38.4" extent="1-16" drill="0.5"/>
 <via x="9.15" y="12.3" extent="1-16" drill="0.5"/>
+<via x="2.85" y="12.2" extent="1-16" drill="0.5"/>
+<via x="2.7" y="2.2" extent="1-16" drill="0.5"/>
+<via x="9.2" y="2.1" extent="1-16" drill="0.5"/>
+<via x="16.7" y="1.9" extent="1-16" drill="0.5"/>
+<via x="23.9" y="1.9" extent="1-16" drill="0.5"/>
+<via x="30.25" y="1.7" extent="1-16" drill="0.5"/>
+<via x="37.35" y="1.9" extent="1-16" drill="0.5"/>
+<via x="43.95" y="1.9" extent="1-16" drill="0.5"/>
+<via x="6.1" y="33.65" extent="1-16" drill="0.5"/>
+<via x="10.65" y="35.05" extent="1-16" drill="0.5"/>
+<via x="38.65" y="33.6" extent="1-16" drill="0.5"/>
+<via x="45.85" y="32.9" extent="1-16" drill="0.5"/>
+<via x="42.85" y="47.25" extent="1-16" drill="0.5"/>
+<via x="12" y="46.6" extent="1-16" drill="0.5"/>
+<via x="2" y="48.65" extent="1-16" drill="0.5"/>
+<via x="2.1" y="35.8" extent="1-16" drill="0.5"/>
+<via x="6.1" y="27.45" extent="1-16" drill="0.5"/>
+<via x="6.1" y="14.55" extent="1-16" drill="0.5"/>
+<via x="39.1" y="12.65" extent="1-16" drill="0.5"/>
+<via x="47.6" y="47.9" extent="1-16" drill="0.5"/>
+<via x="4.2" y="38.4" extent="1-16" drill="0.5"/>
+<via x="12.65" y="38.5" extent="1-16" drill="0.5"/>
+<via x="15.75" y="41" extent="1-16" drill="0.5"/>
+<via x="12.3" y="41.4" extent="1-16" drill="0.5"/>
+<via x="45.85" y="30.35" extent="1-16" drill="0.5"/>
+<via x="36.9" y="27.8" extent="1-16" drill="0.5"/>
+<via x="34.25" y="25.95" extent="1-16" drill="0.5"/>
+<via x="43.1" y="13.95" extent="1-16" drill="0.5"/>
+<via x="31.8" y="11.25" extent="1-16" drill="0.5"/>
+<via x="23.3" y="13.7" extent="1-16" drill="0.5"/>
+<via x="9.3" y="30.2" extent="1-16" drill="0.5"/>
+<via x="19.6" y="30.8" extent="1-16" drill="0.5"/>
+<via x="37.8" y="38.65" extent="1-16" drill="0.5"/>
+<via x="24.95" y="21.9" extent="1-16" drill="0.5"/>
+<via x="22.55" y="20.6" extent="1-16" drill="0.5"/>
+<via x="39.5" y="8.1" extent="1-16" drill="0.5"/>
+<via x="39.15" y="17.55" extent="1-16" drill="0.5"/>
 </signal>
 <signal name="VCC">
